Commit message: Add hand_visualization package

File: catkin_ws/src/my_urdf_test_pkg/urdf/my_simple_model.urdf (robot description, URDF)
Before this commit: robot my_simple_model, 3 links, 2 joints
Links:
- removed link base_link
- removed link l1
- removed link world
- added link link1; visual mesh filename=package://my_urdf_test_pkg/meshes/test_re.stl
Joints:
- removed joint base_joint
- removed joint j1
